File: Keyboard V2.kicad_pcb (KiCad board)
At the start: 2 copper layers, 393.6 x 133 mm, 309 parts, among them J2 Conn_01x04, J3 Conn_01x02, SW1 SW_Push, SW10 SW_Push, SW11 SW_Push, SW12 SW_Push, SW13 SW_Push, SW14 SW_Push, SW15 SW_Push, SW16 SW_Push, SW17 SW_Push, SW18 SW_Push, SW19 SW_Push, SW2 SW_Push, SW20 SW_Push, SW21 SW_Push, SW22 SW_Push, SW23 SW_Push, SW24 SW_Push, SW25 SW_Push, SW26 SW_Push, SW27 SW_Push, SW28 SW_Push, SW29 SW_Push, SW3 SW_Push, SW30 SW_Push, SW31 SW_Push, SW32 SW_Push, SW33 SW_Push, SW34 SW_Push, SW35 SW_Push, SW36 SW_Push, SW37 SW_Push, SW38 SW_Push, SW39 SW_Push, SW4 SW_Push, SW40 SW_Push, SW41 SW_Push, SW42 SW_Push, SW43 SW_Push, SW44 SW_Push, SW45 SW_Push, SW46 SW_Push, SW47 SW_Push, SW48 SW_Push, SW49 SW_Push, SW5 SW_Push, SW50 SW_Push, SW51 SW_Push, SW52 SW_Push, SW53 SW_Push, SW54 SW_Push, SW55 SW_Push, SW56 SW_Push, SW57 SW_Push, SW58 SW_Push, SW59 SW_Push, SW6 SW_Push, SW60 SW_Push, SW61 SW_Push, SW62 SW_Push, SW63 SW_Push, SW64 SW_Push, SW65 SW_Push, SW66 SW_Push, SW67 SW_Push, SW68 SW_Push, SW69 SW_Push, SW7 SW_Push, SW70 SW_Push, SW71 SW_Push, SW72 SW_Push, SW73 SW_Push, SW74 SW_Push, SW75 SW_Push, SW76 SW_Push, SW77 SW_Push, SW78 SW_Push, SW79 SW_Push, SW8 SW_Push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

Commit message: Final board: nano on back, all nets routed, new gerbers/drills/STEP (2026-10-18)
Co-Authored-By: Claude Sonnet 5.5 <noreply@anthropic.com>
Claude-Session: https://claude.ai/code/session_01Mxb6JZ3vXwb4Er3iwwbvVW
Parts:
- U2: moved to B.Cu
- moved D97 4.76 mm to (382.3, 312.0)
- moved LED97 4.76 mm to (391.0, 310.6)
- moved SW97 4.76 mm to (391.0, 306.0)
- moved D85 4.76 mm to (363.2, 293.0)
- moved D95 4.76 mm to (344.2, 312.0)
- moved D96 4.76 mm to (363.2, 312.0)
- moved LED85 4.76 mm to (372.0, 291.6)
- moved LED95 4.76 mm to (352.9, 310.6)
- moved LED96 4.76 mm to (372.0, 310.6)
- moved SW85 4.76 mm to (372.0, 287.0)
- moved SW95 4.76 mm to (352.9, 306.0)
- moved SW96 4.76 mm to (372.0, 306.0)
- turned J3 to 180 degrees
- turned U2 to 180 degrees
- renumbered G*** to G1, G*** to G2
Connections:
- LED12 pad 4: /CHAIN3 -> /CHAIN2
- LED13 pad 2: /CHAIN3 -> /CHAIN2
- LED2 pad 4: /CHAIN3 -> /CHAIN1
- LED3 pad 2: /CHAIN3 -> /CHAIN1
- LED32 pad 4: /CHAIN3 -> /CHAIN4
- LED33 pad 2: /CHAIN3 -> /CHAIN4
- LED42 pad 4: /CHAIN3 -> /CHAIN5
- LED43 pad 2: /CHAIN3 -> /CHAIN5
- LED52 pad 4: /CHAIN3 -> /CHAIN6
- LED53 pad 2: /CHAIN3 -> /CHAIN6
- LED62 pad 4: /CHAIN3 -> /CHAIN7
- LED63 pad 2: /CHAIN3 -> /CHAIN7
- LED72 pad 4: /CHAIN3 -> /CHAIN8
- LED73 pad 2: /CHAIN3 -> /CHAIN8
- LED82 pad 4: /CHAIN3 -> /CHAIN9
- LED83 pad 2: /CHAIN3 -> /CHAIN9
- LED92 pad 4: /CHAIN3 -> /CHAIN10
- LED93 pad 2: /CHAIN3 -> /CHAIN10
- SW97 pad 2: unconnected-(SW97-Pad2) -> /COL7
Routing:
- net /CHAIN3: track 935.2 -> 15.7 mm, vias 30 -> 0
- net /CHAIN6: track 0.00 -> 472.3 mm, vias 0 -> 2
- net /COL7: track 860.5 -> 1054.9 mm, vias 15 -> 20
- net /CHAIN10: track 0.00 -> 114.9 mm, vias 0 -> 2
- net /BAT-: track 150.5 -> 243.4 mm, vias 4 -> 1
- net /LED_DATA: track 386.7 -> 446.2 mm, vias 3 -> 2
- net /COL8: track 844.1 -> 786.1 mm, vias 12 -> 7
- net /COL4: track 877.6 -> 830.7 mm
- net /ROW10: track 342.5 -> 303.1 mm
- net /COL2: track 903.9 -> 873.3 mm, vias 12 -> 9
- net /I2C_SDA: track 170.9 -> 200.6 mm
- net /COL3: track 921.8 -> 896.2 mm, vias 12 -> 9
- net /ROW9: track 555.4 -> 534.4 mm, vias 3 -> 2
- net /COL5: track 901.9 -> 920.5 mm, vias 24 -> 28
- net /ROW1: track 399.3 -> 417.7 mm
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